File: board.kicad_sch (KiCad schematic)
At the start: 26 parts, among them J1 GB_Cart_Edge_32, U1 SST39SF040, U2 FM18W08, U3 74HC574, U4 74HC32, U5 74HC32, U6 74HC00

Commit message: Route the board with Freerouting; JLC part fields and order files
- Fully routed 2-layer board (134/134 connections) from fabdesk's route_run
  with Freerouting 2.4.1; DRC 0 errors / 0 unconnected, ERC clean. Placement
  tweaks (U2, U3, C2, C3, C6, R2-R6) and rules (0.2 mm track, 0.15 mm
  clearance, 0.5/0.3 mm vias) mirrored in circuit.netlist.json and gen.py.
- MPN / Manufacturer / LCSC on all 19 assembled parts in the board and
  schematic (scripts/sync_fields.py).
- exports/jlcpcb: gerbers.zip, bom.csv, cpl.csv (scripts/jlc_export.py).
- Refreshed GLB/STEP exports, 3D and routing renders, README status.

Co-Authored-By: Claude Opus 5.5 <noreply@anthropic.com>
Claude-Session: https://claude.ai/code/session_01K74FFAntk76NicGJzRejN5
Parts:
- C1, C2, C3, C4, C5, C6: LCSC (none) -> C14663; MPN (none) -> CC0603KRX7R9BB104; Manufacturer (none) -> Yageo
- C7: LCSC (none) -> C13585; MPN (none) -> CL31A106KBHNNNE; Manufacturer (none) -> Samsung
- R1: LCSC (none) -> C25804; MPN (none) -> 0603WAF1002T5E; Manufacturer (none) -> UNI-ROYAL
- R2, R3, R4, R5, R6: LCSC (none) -> C4190; MPN (none) -> 0603WAF2201T5E; Manufacturer (none) -> UNI-ROYAL
- U1: LCSC (none) -> C632847; MPN SST39SF040-70-4C-NHE -> SST39SF040-55-4I-NHE-T
- U2: LCSC (none) -> C55945; MPN FM18W08-SG -> FM18W08-SGTR
- U3: LCSC (none) -> C10097
- U4, U5: LCSC (none) -> C6838
- U6: LCSC (none) -> C10090

Commit message: r1.1: DMG cartridge outline, re-routed, DRC clean
r1 (56 x 49.5 mm) did not fit a cartridge shell. r1.1 is the same circuit on
the OEM outline (51.4 x 61 mm, finger tongue, lock notch, shell holes),
1.0 mm thick, edge fingers 1.5 mm above the board edge.

- Re-placed inside the shell component zone and re-routed in fabdesk with
  Freerouting (134/134), copper keep-outs around both shell holes
- DRC 0 errors / 0 unconnected (silkscreen warnings only); fit check passes
  (PLCC-32 height warning)
- JLC gerbers / CPL, renders and README updated

Co-Authored-By: Claude Opus 5.5 <noreply@anthropic.com>
Claude-Session: https://claude.ai/code/session_01K74FFAntk76NicGJzRejN5
Parts:
- J1: footprint gbdev:GB_Cart_Edge_32 -> gbdev:GB_Cart_Edge_32_DMG
